Commit message: update

File: xacro/r7bot_urdf.xacro (robot description, xacro)
@@ -4,10 +4,4 @@
   <xacro:include filename="$(find r7bot)/xacro/r7bot_description.xacro"/>
   <xacro:include filename="$(find r7bot)/xacro/r7bot_ros2_control.xacro" />
-  <!-- Used for fixing robot -->
-  <link name="world"/>
-  <joint name="pin" type="fixed">
-    <parent link="world"/>
-    <child link="base_link"/>
-  </joint>
   <!-- Use macros -->
   <xacro:r7bot_description/>
